File: Hardware/stm32f103-ibus.sch (KiCad schematic (older format))
At the start: 60 parts, among them IC1 PC817, IC2 PC817, IC3 PC817, IC4 PC817, K1 SANYOU_SRD_Form_C, P1 USART2, P2 POWER, P3 I-Bus, P4 D-Bus, P5 HEATER, P6 PWM_FAN, P7 SWD, Q1 S8050, Q2 S8050, Q3 S8050, Q4 S8050, Q5 S8050, Q6 S8050, Q7 S8050, SW1 SW_PUSH, U1 LM358N, U2 STM32F103C(8-B)Tx, Y1 8M, Y2 32.768K

Commit message: Various update 1.Optimization of compiler options 2.Supports internal flash read / write 3.Supports 1999 model
Parts:
- C1, C2, C3, C4, C5, C6, C7, C8, C9: symbol C -> stm32f103-ibus-rescue:C
- D1, D2: symbol LED -> stm32f103-ibus-rescue:LED
- D3: symbol 1N4148 -> stm32f103-ibus-rescue:1N4148
- IC1, IC2, IC3, IC4: symbol PC817-RESCUE-stm32f103-ibus -> stm32f103-ibus-rescue:PC817-RESCUE-stm32f103-ibus
- K1: symbol SANYOU_SRD_Form_C -> stm32f103-ibus-rescue:SANYOU_SRD_Form_C
- P1, P7: symbol CONN_01X04 -> stm32f103-ibus-rescue:CONN_01X04
- P2: symbol CONN_01X02 -> stm32f103-ibus-rescue:CONN_01X02
- P3, P4, P5, P6: symbol CONN_01X01 -> stm32f103-ibus-rescue:CONN_01X01
- Q1, Q2, Q3, Q4, Q5, Q6, Q7: symbol S8050 -> stm32f103-ibus-rescue:S8050
- R1, R10, R11, R13, R14, R15, R16, R17, R18, R6, R7, R8, R9: symbol R-RESCUE-stm32f103-ibus -> stm32f103-ibus-rescue:R-RESCUE-stm32f103-ibus
- R12, R19, R2, R20, R22, R23, R24, R25, R3, R4, R5: symbol R -> stm32f103-ibus-rescue:R
- SW1: symbol SW_PUSH -> stm32f103-ibus-rescue:SW_PUSH
- U1: symbol LM358N -> stm32f103-ibus-rescue:LM358N
- U2: symbol STM32F103C(8-B)Tx -> stm32f103-ibus-rescue:STM32F103C(8-B)Tx
- Y1, Y2: symbol Crystal -> stm32f103-ibus-rescue:Crystal
